File: isolator.kicad_pcb (KiCad board)
At the start: 4 copper layers, 120 x 75 mm, 125 parts, among them J1 HOST, J2 USB_C_Receptacle_PowerOnly_6P, J3 USB_A, J4 USB_A, J5 USB_C_Receptacle_USB2.0_16P, J6 USB_C_Receptacle_USB2.0_16P, Q1 2N7002, Q2 2N7002, T1 750313638, U1 ADuM4165, U10 TPS2553DBV, U11 TPS2553DBV, U12 TPS2553DBV, U13 TLV7041DBV, U14 TLV7041DBV, U15 USBLC6-2SC6, U16 USBLC6-2SC6, U17 USBLC6-2SC6, U18 USBLC6-2SC6, U2 USBLC6-2SC6, U3 USBLC6-2SC6, U4 USB2514B_Bi, U5 SN6505BDBV, U6 MIC29302WU, U7 TPS2121, U8 AP2112K-3.3, U9 TPS2553DBV, Y1 24M 8pF, Y2 24M 12pF

Commit message: fix(pcb): rotate U3 180° and shift 0.6 mm west so the ISO_D pair does not cross
U3 (ISO-side USBLC6-2SC6) sat at rot 0, which put ISO_D+/ISO_D- in the
opposite order to BOTH neighbours:

  U1  pad12 = ISO_D+ (y 75.445), pad13 = ISO_D- (y 74.175)   -> D- north
  U3  pad1  = ISO_D+ (y 72.05),  pad3  = ISO_D- (y 73.95)    -> D- south
  U4  pad31 = ISO_D+ (x 116.5),  pad30 = ISO_D- (x 117.0)    -> D- east

A differential pair cannot swap members without a layer crossunder, so the
old orientation cost two crossunders (4 vias) on the isolated high-speed
link — one between U1 and U3 and another between U3 and U4.  Rotating U3
180° makes the member order agree at both ends, so the pair runs with zero
intra-pair crossings.

The extra 0.6 mm west shift keeps U3's new GND2 pad clear of the existing
/ISO_5V stitching via at (101.125, 73.0), which the un-shifted rotation
would have left 0.025 mm away.

No copper was attached to U3, so nothing else moves.

Co-Authored-By: Claude Fable 5 <noreply@anthropic.com>
Parts:
- moved U3 0.60 mm to (98.4, 73.0), turned to 180 degrees
Changed lines of the file:
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@@
 	(footprint "Package_TO_SOT_SMD:SOT-23-6"
 		(layer "F.Cu")
-		(at 99 73)
+		(at 98.4 73 180)
 		(descr "SOT, 6 Pin (JEDEC MO-178 Var AB https://www.jedec.org/document_search?search_api_views_fulltext=MO-178)")
 		(tags "SOT TO_SOT_SMD")
 		(property "Reference" "U3"
-			(at 0 -2.4 0)
+			(at 0 -2.4 180)
 			(layer "F.SilkS")
 			(effects
@@
 		)
 		(property "Value" "USBLC6-2SC6"
-			(at 0 2.4 0)
+			(at 0 2.4 180)
 			(layer "F.Fab")
 			(effects
@@
 		)
 		(property "Datasheet" "https://www.st.com/resource/en/datasheet/usblc6-2.pdf"
-			(at 0 0 0)
+			(at 0 0 180)
 			(layer "F.Fab")
 			(hide yes)
@@
 		)
 		(property "Description" "Very low capacitance ESD protection diode, 2 data-line, SOT-23-6"
-			(at 0 0 0)
+			(at 0 0 180)
 			(layer "F.Fab")
 			(hide yes)
@@
 		)
 		(property "KiLib_Generator" "package/gullwing"
-			(at 0 0 0)
+			(at 0 0 180)
 			(layer "F.SilkS")
 			(hide yes)
@@
 		)
 		(property "MPN" "USBLC6-2SC6"
-			(at 0 0 0)
+			(at 0 0 180)
 			(unlocked yes)
 			(layer "F.Fab")
@@
 		)
 		(property "Manufacturer" "STMicroelectronics"
-			(at 0 0 0)
+			(at 0 0 180)
 			(unlocked yes)
 			(layer "F.Fab")
@@
 		)
 		(property "LCSC" "C2687116"
-			(at 0 0 0)
+			(at 0 0 180)
 			(unlocked yes)
 			(layer "F.Fab")
@@
 		(duplicate_pad_numbers_are_jumpers no)
 		(fp_line
+			(start 0.91 1.56)
+			(end -0.91 1.56)
+			(stroke
+				(width 0.12)
+				(type solid)
+			)
+			(layer "F.SilkS")
+		)
+		(fp_line
+			(start 0.91 1.51)
+			(end 0.91 1.56)
+			(stroke
+				(width 0.12)
+				(type solid)
+			)
+			(layer "F.SilkS")
+		)
+		(fp_line
+			(start 0.91 -1.56)
+			(end 0.91 -1.51)
+			(stroke
+				(width 0.12)
+				(type solid)
+			)
+			(layer "F.SilkS")
+		)
+		(fp_line
+			(start -0.91 1.56)
+			(end -0.91 1.51)
+			(stroke
+				(width 0.12)
+				(type solid)
+			)
+			(layer "F.SilkS")
+		)
+		(fp_line
+			(start -0.91 -1.51)
+			(end -0.91 -1.56)
+			(stroke
+				(width 0.12)
+				(type solid)
+			)
+			(layer "F.SilkS")
+		)
+		(fp_line
 			(start -0.91 -1.56)
 			(end 0.91 -1.56)
-			(stroke
-				(width 0.12)
-				(type solid)
-			)
-			(layer "F.SilkS")
-		)
-		(fp_line
-			(start -0.91 -1.51)
-			(end -0.91 -1.56)
-			(stroke
-				(width 0.12)
-				(type solid)
-			)
-			(layer "F.SilkS")
-		)
-		(fp_line
-			(start -0.91 1.56)
-			(end -0.91 1.51)
-			(stroke
-				(width 0.12)
-				(type solid)
-			)
-			(layer "F.SilkS")
-		)
-		(fp_line
-			(start 0.91 -1.56)
-			(end 0.91 -1.51)
-			(stroke
-				(width 0.12)
-				(type solid)
-			)
-			(layer "F.SilkS")
-		)
-		(fp_line
-			(start 0.91 1.51)
-			(end 0.91 1.56)
-			(stroke
-				(width 0.12)
-				(type solid)
-			)
-			(layer "F.SilkS")
-		)
-		(fp_line
-			(start 0.91 1.56)
-			(end -0.91 1.56)
 			(stroke
 				(width 0.12)
@@
 		)
 		(fp_line
+			(start 2.05 1.5)
+			(end 1.05 1.5)
+			(stroke
+				(width 0.05)
+				(type solid)
+			)
+			(layer "F.CrtYd")
+		)
+		(fp_line
+			(start 2.05 -1.5)
+			(end 2.05 1.5)
+			(stroke
+				(width 0.05)
+				(type solid)
+			)
+			(layer "F.CrtYd")
+		)
+		(fp_line
+			(start 1.05 1.7)
+			(end -1.05 1.7)
+			(stroke
+				(width 0.05)
+				(type solid)
+			)
+			(layer "F.CrtYd")
+		)
+		(fp_line
+			(start 1.05 1.5)
+			(end 1.05 1.7)
+			(stroke
+				(width 0.05)
+				(type solid)
+			)
+			(layer "F.CrtYd")
+		)
+		(fp_line
+			(start 1.05 -1.5)
+			(end 2.05 -1.5)
+			(stroke
+				(width 0.05)
+				(type solid)
+			)
+			(layer "F.CrtYd")
+		)
+		(fp_line
+			(start 1.05 -1.7)
+			(end 1.05 -1.5)
+			(stroke
+				(width 0.05)
+				(type solid)
+			)
+			(layer "F.CrtYd")
+		)
+		(fp_line
+			(start -1.05 1.7)
+			(end -1.05 1.5)
+			(stroke
+				(width 0.05)
+				(type solid)
+			)
+			(layer "F.CrtYd")
+		)
+		(fp_line
+			(start -1.05 1.5)
+			(end -2.05 1.5)
+			(stroke
+				(width 0.05)
+				(type solid)
+			)
+			(layer "F.CrtYd")
+		)
+		(fp_line
+			(start -1.05 -1.5)
+			(end -1.05 -1.7)
+			(stroke
+				(width 0.05)
+				(type solid)
+			)
+			(layer "F.CrtYd")
+		)
+		(fp_line
+			(start -1.05 -1.7)
+			(end 1.05 -1.7)
+			(stroke
+				(width 0.05)
+				(type solid)
+			)
+			(layer "F.CrtYd")
+		)
+		(fp_line
+			(start -2.05 1.5)
+			(end -2.05 -1.5)
+			(stroke
+				(width 0.05)
+				(type solid)
+			)
+			(layer "F.CrtYd")
+		)
+		(fp_line
 			(start -2.05 -1.5)
 			(end -1.05 -1.5)
-			(stroke
-				(width 0.05)
-				(type solid)
-			)
-			(layer "F.CrtYd")
-		)
-		(fp_line
-			(start -2.05 1.5)
-			(end -2.05 -1.5)
-			(stroke
-				(width 0.05)
-				(type solid)
-			)
-			(layer "F.CrtYd")
-		)
-		(fp_line
-			(start -1.05 -1.7)
-			(end 1.05 -1.7)
-			(stroke
-				(width 0.05)
-				(type solid)
-			)
-			(layer "F.CrtYd")
-		)
-		(fp_line
-			(start -1.05 -1.5)
-			(end -1.05 -1.7)
-			(stroke
-				(width 0.05)
-				(type solid)
-			)
-			(layer "F.CrtYd")
-		)
-		(fp_line
-			(start -1.05 1.5)
-			(end -2.05 1.5)
-			(stroke
-				(width 0.05)
-				(type solid)
-			)
-			(layer "F.CrtYd")
-		)
-		(fp_line
-			(start -1.05 1.7)
-			(end -1.05 1.5)
-			(stroke
-				(width 0.05)
-				(type solid)
-			)
-			(layer "F.CrtYd")
-		)
-		(fp_line
-			(start 1.05 -1.7)
-			(end 1.05 -1.5)
-			(stroke
-				(width 0.05)
-				(type solid)
-			)
-			(layer "F.CrtYd")
-		)
-		(fp_line
-			(start 1.05 -1.5)
-			(end 2.05 -1.5)
-			(stroke
-				(width 0.05)
-				(type solid)
-			)
-			(layer "F.CrtYd")
-		)
-		(fp_line
-			(start 1.05 1.5)
-			(end 1.05 1.7)
-			(stroke
-				(width 0.05)
-				(type solid)
-			)
-			(layer "F.CrtYd")
-		)
-		(fp_line
-			(start 1.05 1.7)
-			(end -1.05 1.7)
-			(stroke
-				(width 0.05)
-				(type solid)
-			)
-			(layer "F.CrtYd")
-		)
-		(fp_line
-			(start 2.05 -1.5)
-			(end 2.05 1.5)
-			(stroke
-				(width 0.05)
-				(type solid)
-			)
-			(layer "F.CrtYd")
-		)
-		(fp_line
-			(start 2.05 1.5)
-			(end 1.05 1.5)
 			(stroke
 				(width 0.05)
@@
 		)
 		(fp_text user "${REFERENCE}"
-			(at 0 0 90)
+			(at 0 0 270)
 			(layer "F.Fab")
 			(effects
@@
 		)
 		(pad "1" smd roundrect
-			(at -1.1375 -0.95)
+			(at -1.1375 -0.95 180)
 			(size 1.325 0.6)
 			(layers "F.Cu" "F.Mask" "F.Paste")
@@
 		)
 		(pad "2" smd roundrect
-			(at -1.1375 0)
+			(at -1.1375 0 180)
 			(size 1.325 0.6)
 			(layers "F.Cu" "F.Mask" "F.Paste")
@@
 		)
 		(pad "3" smd roundrect
-			(at -1.1375 0.95)
+			(at -1.1375 0.95 180)
 			(size 1.325 0.6)
 			(layers "F.Cu" "F.Mask" "F.Paste")
@@
 		)
 		(pad "4" smd roundrect
-			(at 1.1375 0.95)
+			(at 1.1375 0.95 180)
 			(size 1.325 0.6)
 			(layers "F.Cu" "F.Mask" "F.Paste")
@@
 		)
 		(pad "5" smd roundrect
-			(at 1.1375 0)
+			(at 1.1375 0 180)
 			(size 1.325 0.6)
 			(layers "F.Cu" "F.Mask" "F.Paste")
@@
 		)
 		(pad "6" smd roundrect
-			(at 1.1375 -0.95)
-			(size 1.325 0.6)
-			(layers "F.Cu" "F.Mask" "F.Paste")
+			(at 1.1375 -0.95 180)
+			(size 1.325 0.6)
+			(layers "F.Cu" "F.Mask" "F.Paste")

Commit message: feat(pcb): route cluster-local nets
22 short two/three-point nets whose pads all sit within ~9 mm of each other,
routed on F.Cu with 45/90 geometry only, 0.20 mm width, no vias:

  ILIM sense      /P1_ILIM /P2_ILIM /P3_ILIM /P4_ILIM /ILIM_SET
  hub straps      /HUB_CFG_SEL0 /HUB_CFG_SEL1 /HUB_NON_REM0 /HUB_NON_REM1
  hub analog      /HUB_RBIAS /HUB_CRFILT /HUB_PLLFILT /HUB_XO
  soft start      /SS_SET
  regulator ADJ   Net-(U6-ADJ)
  USB-C CC        /P3_CC1 /P4_CC1 /P4_CC2
  indicators      /ST_LED /PGOOD_LED_A /PGOOD_LED_K /DCDC_LED_A

Every candidate path was walked against an exact clearance model (rotated-rect
pads, capsule tracks, circular vias; 0.15 mm inter-net clearance, 0.30 mm to
the board edge) before being accepted.

Skipped: /VDD2 (U1.18 -> C36.1) - U1's pad 18 escape is boxed in by the
existing GND2 stitching stubs at (93.4, 69.095) and (93.4, 71.635).

DRC: unconnected 194 -> 170, no new violation types, shorting 0, dangling 0.

Co-Authored-By: Claude Fable 5 <noreply@anthropic.com>
Routing:
- net /HUB_XO: track 0.00 -> 12.8 mm
- net /P4_CC2: track 0.00 -> 8.88 mm
- net /PGOOD_LED_K: track 0.00 -> 7.98 mm
- net Net-(U6-ADJ): track 0.00 -> 6.10 mm
- net /HUB_PLLFILT: track 0.00 -> 5.69 mm
- net /HUB_NON_REM1: track 0.00 -> 5.62 mm
- net /HUB_CFG_SEL1: track 0.00 -> 5.41 mm
- net /HUB_CFG_SEL0: track 0.00 -> 5.41 mm
- net /P4_CC1: track 0.00 -> 4.17 mm
- net /P3_CC1: track 0.00 -> 4.17 mm
- net /P4_ILIM: track 0.00 -> 3.39 mm
- net /P3_ILIM: track 0.00 -> 3.39 mm
- net /HUB_RBIAS: track 0.00 -> 3.02 mm
- net /HUB_NON_REM0: track 0.00 -> 3.02 mm
- net /SS_SET: track 0.00 -> 1.96 mm
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