File: hub.kicad_sch (KiCad schematic)
At the start: 105 parts, among them J1 USB_C_Receptacle_USB2.0_16P, J2 USB_C_Receptacle_PowerOnly_6P, Q1 2N7002, Q2 2N7002, Q3 2N7002, Q4 2N7002, T1 750313638, U1 ADuM4165, U10 TPS62203DBVR, U11 USB2514B, U2 USBLC6-2SC6, U3 TLV7042DDFR, U5 SN6505BDBV, U6 TPS630701RNM, U7 TLV7042DDFR, U8 TPS2121, Y1 24MHz, Y2 24MHz

Commit message: feat(revb/sch): assign footprints to all 105 hub components
Lifts the shared assignments from rev A (ADuM4165, 750313638, USB-C host
receptacle, USBLC6, SN6505B, crystals, SS34, SOD-523 TVS) and resolves the
rev B-only parts against the part-selection decision record:

- U3/U7 TLV7042DDFR -> SOT-23-8 (DDF)
- U8  TPS2121       -> Texas_VQFN-HR-12_2x2.5mm_P0.5mm (RUX0012A)
- U6  TPS630701RNM  -> isolator-lib:TPS630701RNM_VQFN-HR-15
- U10 TPS62203DBVR  -> SOT-23-5 (DBV), pin-compatible with the AP2112K option
- U11 USB2514B      -> QFN-36-1EP_6x6mm_P0.5mm_EP3.7x3.7mm
- J2  power-only    -> GCT USB4125 6P top-mount (3 A)
- L1  XFL4020-152MEC -> L_Coilcraft_XxL4020
- L2  744043100      -> L_Wuerth_WE-PD-Typ-M-Typ-S

Passives follow the decision record's ordered parts: 0402 for resistors and
for ceramics <= 1 uF, 0805 for 4.7/10/22 uF, 1210 for the 47 uF rectifier
bulk.

Netlist unchanged: 91 nets, 105 components, identical membership.

Co-Authored-By: Claude Opus 5 <noreply@anthropic.com>
Parts:
- C1, C10, C12, C14, C17, C21, C22, C23, C25, C26, C27, C28, C29, C3, C32, C33, C34, C35, C36, C37, C38, C39, C4, C40, C42, C5, C6, C7, C8: footprint (none) -> Capacitor_SMD:C_0402_1005Metric
- C11, C15, C16, C18, C19, C2, C20, C24, C30, C31, C41: footprint (none) -> Capacitor_SMD:C_0805_2012Metric
- C13: footprint (none) -> Capacitor_SMD:C_1210_3225Metric
- D1, D5: footprint (none) -> Diode_SMD:D_SOD-523
- D2, D6, D7: footprint (none) -> LED_SMD:LED_0603_1608Metric
- D3, D4: footprint (none) -> Diode_SMD:D_SMA
- J1: footprint (none) -> Connector_USB:USB_C_Receptacle_HRO_TYPE-C-31-M-12
- J2: footprint (none) -> Connector_USB:USB_C_Receptacle_GCT_USB4125-xx-x_6P_TopMnt_Horizontal
- L1: footprint (none) -> Inductor_SMD:L_Coilcraft_XxL4020
- L2: footprint (none) -> Inductor_SMD:L_Wuerth_WE-PD-Typ-M-Typ-S
- Q1, Q2, Q3, Q4: footprint (none) -> Package_TO_SOT_SMD:SOT-23
- R1, R10, R11, R12, R13, R14, R15, R16, R17, R18, R19, R2, R20, R21, R22, R23, R24, R25, R26, R27, R28, R29, R3, R30, R31, R32, R33, R34, R35, R36, R37, R4, R5, R6, R7, R8, R9: footprint (none) -> Resistor_SMD:R_0402_1005Metric
- U1: footprint (none) -> isolator-lib:ADI_SOIC_IC_20_RI-20-1
- U10: footprint (none) -> Package_TO_SOT_SMD:SOT-23-5
- U11: footprint (none) -> Package_DFN_QFN:QFN-36-1EP_6x6mm_P0.5mm_EP3.7x3.7mm
- U2, U5: footprint (none) -> Package_TO_SOT_SMD:SOT-23-6
- U3, U7: footprint (none) -> Package_TO_SOT_SMD:SOT-23-8
- U6: footprint (none) -> isolator-lib:TPS630701RNM_VQFN-HR-15
- U8: footprint (none) -> Package_DFN_QFN:Texas_VQFN-HR-12_2x2.5mm_P0.5mm
- Y1, Y2: footprint (none) -> Crystal:Crystal_SMD_3225-4Pin_3.2x2.5mm

Commit message: refactor(revb/sch): relocate the external-supply and TPS2121 mux blocks
Both were jammed into the 40 mm top strip while the right third of the A3
sheet sat empty. Task 6 (J2, 3 A detect, U7) moves to x 302-398, y 15-55;
the TPS2121 mux moves to x 221-287, y 15-51. Their long design notes are
re-wrapped and parked under the Task 6 block instead of lying across it.

Rigid translation: every symbol moved to an exact coordinate (the bulk-move
tools snap to the 1.27 mm grid, which would detach the sheet's many off-grid
wire endpoints), wires deleted and re-added at the translated coordinates,
junctions re-established, labels moved.

Netlist unchanged (91 nets, identical membership); ERC unchanged at 253
violations across all severities.

Co-Authored-By: Claude Opus 5 <noreply@anthropic.com>
Other:
- note added: "CP2 rule (Table 9-3): CP2=hi,PR1=lo selects IN2; CP2=PR1=lo selects VCOMP (higher wins)."
- note added: "CP2(pin3)=STATIC bias from ISO_5V_PRE, 23.7k/10.2k to GND2, never the 3A detect."
- note added: "PR1(pin6)=driven by the 3A-detect 2N7002 inverter, 17.8k/10.0k EXT_5V to GND2."
- note added: "Switchback: approx 4.18V nominal, worst-case 3.92-4.54V -- measure at bring-up."
- note added: "Task 6: External supply, 3A detect (GND2)"
- note removed: "CP2 rule (Table 9-3): CP2=hi,PR1=lo selects IN2; CP2=PR1=lo selects VCOMP (higher wins). CP2(pin3)=STATIC bias from ISO_5V_PRE, 23.7k/10.2k to GND2, never the 3A detect."
- note removed: "PR1(pin6)=driven by 3A-detect 2N7002 inverter, 17.8k/10.0k EXT_5V to GND2. Switchback: approx 4.18V nominal, worst-case 3.92-4.54V -- measure at bring-up."
- note removed: "Task 6: External supply, 3A detect, TPS2121 priority mux (GND2)"
- moved on the sheet: C23, C24, C25, C26, C27, D5, D6, J2, Q3, R16, R17, R18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

Commit message: fix(revb/sch): zero text overlaps — spread the sheet and re-place every field
Layout-only pass over hub.kicad_sch. Text overlaps go from 220 to 0 and the
last off-page item is gone.

- Spread the decoupling-cap banks: the six-cap DCDC_RAW/ISO_5V_PRE row split
  into an input bank and an output bank; C13/C14, C10, C3/C4, C23/C24 pulled
  apart. These are pin-stacked islands with no wires, so they translate
  safely.
- Staggered the CC pulldowns under J2 and dropped R12 clear of R11 in the
  converter's DNP-divider corner, re-routing the three affected wires.
- Re-placed all 215 symbols' Reference/Value fields with a solver that keeps
  each label within 9.5 mm of its own part, honours the 2.54 mm pair rule and
  1.27 mm general clearance, and treats symbol bodies and wires as obstacles.
- Staggered the PORT_D-/PRTPWR1 label pairs off the 2.54 mm pin pitch, and
  moved U11's GND2 label from below the frame onto its pin.

tools/check_sch_text_overlap.py: a field's stored angle is relative to its
symbol's rotation — KiCad draws it at the sum. The checker treated the stored
angle as absolute, so every rotated part's label box was computed 90 degrees
out. That both hid real collisions (15 of them here) and invented false ones.

Netlist unchanged throughout: 91 nets, 105 components, identical membership;
isolation check clean. ERC 253 -> 225 at --severity-all, the whole delta being
off-grid endpoint warnings that the cap moves cleaned up.

Co-Authored-By: Claude Opus 5 <noreply@anthropic.com>
Other:
- note added: "TPS2121 priority mux (GND2)"
- moved on the sheet: C10, C13, C14, C15, C17, C18, C19, C20, C21, C23, C24, C26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

Commit message: refactor(revb/sch): A2 re-flow — boxed sections, wide gulfs, all-orthogonal wiring
Alex: the A3 sheet was 72% full and unreadable. Changes:

- Paper A3 -> A2. Eight functional blocks rigidly translated apart with
  30-100 mm gulfs between them, in signal-flow order: host -> isolation ->
  CC sense on the top row, mux/external supply top-right, isolated power ->
  3.3V rail -> hub across the bottom. All moves netlist-gated.
- Every diagonal wire (9) redrawn as Manhattan H/V routes: the D6/R28/R29
  status-LED tangle, the R18/R19/C25 divider (which also had a wire ending
  inside R18's body), R21->U7.6, the RESET_N_HUB label stub, and the Y2
  crystal fan-out, which previously ran a diagonal straight through the
  crystal body.
- Dashed section boxes (rev A style, 0.254 dash) around all eight blocks
  with bold uppercase titles; the four scattered task-title texts replaced,
  design-note paragraphs parked under their owning boxes.
- Block deltas snapped to 1.27 mm multiples (first pass used integer mm and
  pushed every moved endpoint off the connection grid; ERC off-grid count
  is now 153, below the 186 baseline).
- Field placer taught about box edges; residual field/label collisions
  cleaned. Both overlap checkers report zero; no diagonals remain.

Netlist identical throughout: 91 nets, 105 components, same membership;
isolation check clean. ERC 253 -> 219 at --severity-all (all improvement,
no new violations).

Co-Authored-By: Claude Opus 5 <noreply@anthropic.com>
Other:
- note added: "3.3V RAIL (GND2)"
- note added: "EXTERNAL SUPPLY + 3A DETECT (GND2)"
- note added: "ISOLATED POWER - SN6505B + TPS630701 (GND1 | GND2)"
- note added: "TPS2121 SUPPLY PRIORITY MUX (GND2)"
- note added: "UPSTREAM CC CURRENT-ADVERTISEMENT SENSE (GND1)"
- note added: "USB ISOLATION - ADuM4165 (GND1 | GND2)"
- note added: "USB2514B 4-PORT HUB (GND2)"
- note removed: "TPS2121 priority mux (GND2)"
- note removed: "Task 4: Upstream CC current-advertisement sensing (GND1)"
- note removed: "Task 6: External supply, 3A detect (GND2)"
- moved on the sheet: C1, C10, C11, C12, C13, C14, C15, C16, C17, C18, C19, C2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
