File: hub.kicad_sch (KiCad schematic)
At the start: 105 parts, among them J1 USB_C_Receptacle_USB2.0_16P, J2 USB_C_Receptacle_PowerOnly_6P, Q1 2N7002, Q2 2N7002, Q3 2N7002, Q4 2N7002, T1 750313638, U1 ADuM4165, U10 TPS62203DBVR, U11 USB2514B, U2 USBLC6-2SC6, U3 TLV7042DDFR, U5 SN6505BDBV, U6 TPS630701RNM, U7 TLV7042DDFR, U8 TPS2121, Y1 24MHz, Y2 24MHz

Commit message: feat(revb/sch): Task 8 ports 1-3 — 2x TPS2553 USB-A switches, 1x USB-C w/ CC pull-ups
Port 1 (J3, USB-A) and Port 2 (J4, USB-A) complete: TPS2553DBV switch,
46.4k 1% ILIM (sized from SLVS841F's three threshold equations so
I_OS(min) clears the 500 mA per-port target), USBLC6-2SC6 ESD, TVS,
in/out bypass caps, wired to the hub's PRTPWRn/OCSn/USBDM_DNn/USBDP_DNn
pins.

Port 3 (J5, USB-C) complete: same switch block plus two dedicated 56k
CC pull-ups (never shared, per Default USB Power / rev A brown-out
lesson), D+/D- pinned together across the connector's redundant pads.

Port 4 (J6, USB-C) not yet placed — ran out of contiguous free sheet
area near the other three; needs a placement decision before continuing.

Verified after each port: netlist parse, isolation check (only U1/T1
bridge domains), text-overlap checker (zero new overlaps), and
per-net probes confirming exact expected membership (no shorts).
ERC not yet at zero — expected, Task 9's job.
Parts:
- added C43, C45, C46, C48, C49, C51: 0.1uF, symbol Device:C_Small
- added C44, C47, C50: 22uF, symbol Device:C_Small
- added D10, D8, D9: TVS, symbol Device:D_TVS
- added J3, J4: USB_A, symbol Connector:USB_A
- added J5: USB_C_Receptacle_USB2.0_16P, symbol Connector:USB_C_Receptacle_USB2.0_16P
- added R38, R39, R40: 46.4k 1%, symbol Device:R_Small
- added R42, R43: 56k, symbol Device:R_Small
- added U12, U13, U14: TPS2553DBV, symbol isolator-lib:TPS2553DBV
- added U16, U17, U18: USBLC6-2SC6, symbol Power_Protection:USBLC6-2SC6
Connections:
- net CC_DET_L: now also R5.2, U3.1 (OUTA), U3.7 (OUTB)
- net EXT_5V: now also C25.1, J2.A5 (CC1), R16.1, R18.2, R19.1, R20.1, U7.3 (INA+)
- net GND1: now also C1.2, C2.2
- net GND2: now also C42.2, C43.2, C44.2, C45.2, C46.2, C47.2, C48.2, C49.2, C50.2, C51.2, D10.1 (A1), D8.1 (A1), D9.1 (A1), J3.4 (GND), J3.SH (Shield), J4.4 (GND), J4.SH (Shield), J5.A1 (GND), J5.A12 (GND), J5.B1 (GND), J5.B12 (GND), J5.SH (SHIELD), R38.2, R39.2, R40.2, U12.2 (GND), U13.2 (GND), U14.2 (GND), U16.2 (GND), U17.2 (GND), U18.2 (GND)
- net ISO_5V: now also C43.1, C46.1, C49.1, U12.1 (IN), U13.1 (IN), U14.1 (IN)
- net ISO_5V_PRE: now also R11.2, R12.2, R15.2, U6.1 (PS/SYNC), U6.2 (PG)
- net OCS1: now also U12.4 (~{FAULT})
- net OCS2: now also U13.4 (~{FAULT})
- net OCS3: now also U14.4 (~{FAULT})
- net PRTPWR1: now also U12.3 (EN)
- net PRTPWR2: now also U13.3 (EN)
- net PRTPWR3: now also U14.3 (EN)
- net VBUS_HOST: now also C1.1, C2.1
- net V_REF: now also C7.1, U3.3 (INA+)
- net PORT1_D-: now reaches U11.1 (USBDM_DN1/PRT_DIS_M1)
- net PORT1_D-: now also U16.1 (I/O1)
- net PORT1_D+: now reaches U11.2 (USBDP_DN1/PRT_DIS_P1)
- net PORT1_D+: now also U16.3 (I/O2)
- net PORT2_D-: now reaches U11.3 (USBDM_DN2/PRT_DIS_M2)
- net PORT2_D-: now also U17.1 (I/O1)
- net PORT2_D+: now reaches U11.4 (USBDP_DN2/PRT_DIS_P2)
- net PORT2_D+: now also U17.3 (I/O2)
- net PORT3_D-: now reaches U11.6 (USBDM_DN3/PRT_DIS_M3)
- net PORT3_D-: now also U18.1 (I/O1)
- net PORT3_D+: now reaches U11.7 (USBDP_DN3/PRT_DIS_P3)
- net PORT3_D+: now also U18.3 (I/O2)
- net at R20.2, U7.2 (INA-): now also U7.5 (INB+)
- new net: J5.A5 (CC1), R42.1
- new net: J3.3 (D+), U16.4 (I/O2)
- new net: J3.2 (D-), U16.6 (I/O1)
- new net: J4.2 (D-), U17.6 (I/O1)
- new net: J4.3 (D+), U17.4 (I/O2)
- new net: J5.A6 (D+), J5.B6 (D+), U18.4 (I/O2)
- new net: J5.A7 (D-), J5.B7 (D-), U18.6 (I/O1)
- new net: J5.B5 (CC2), R43.1
- new net ILIM1: R38.1, U12.5 (ILIM)
- new net ILIM2: R39.1, U13.5 (ILIM)
- new net ILIM3: R40.1, U14.5 (ILIM)
- new net PORT1_VBUS: C44.1, C45.1, D8.2 (A2), J3.1 (VBUS), U12.6 (OUT), U16.5 (VBUS)
- new net PORT2_VBUS: C47.1, C48.1, D9.2 (A2), J4.1 (VBUS), U13.6 (OUT), U17.5 (VBUS)
- new net PORT3_VBUS: C50.1, C51.1, D10.2 (A2), J5.A4 (VBUS), J5.A9 (VBUS), J5.B4 (VBUS), J5.B9 (VBUS), R42.2, R43.2, U14.6 (OUT), U18.5 (VBUS)
Other:
- moved on the sheet: C1, C14, C17, C19, C2, C23, C24, C37, C38, C39, C40, C41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

Commit message: feat(revb/sch): Task 8 complete — Port 4 (J6, USB-C) placed and wired
Port 4 needed a compact single-row template in the ~35x130mm pocket
above the design-notes text at bottom-left (x=0-140, y=190-225) — the
only contiguous free area left after ports 1-3 filled the right
column. J6 is rotated 90 deg so its 38mm pin spread runs horizontally
where there's room, instead of vertically where there wasn't.

All four ports now verified structurally identical per net topology:
- PORT{1-4}_VBUS: switch OUT + both bulk caps + TVS + ESD VBUS + every
  physical VBUS pin on the connector (USB-C ports tie 4 redundant
  VBUS pads together automatically — same schematic point).
- PRTPWR{1-4}/OCS{1-4}: exactly {hub pin, switch pin}, 2 nodes each.
- USB-C ports' two 56k Rp resistors verified on dedicated per-CC-pin
  nets, never shared (rev A brown-out lesson).
- D+/D- tied across each USB-C connector's redundant pads, routed
  through the ESD chip to the hub's per-port USBDM/USBDP pins.

Two real bugs surfaced and fixed during routing, worth recording:
one, a straight wire between two pins can pass exactly through a
THIRD unrelated pin sitting on the same line and silently join nets
(hit repeatedly — ILIM resistor placed directly below its switch,
EN/FAULT stubs passing through a neighboring cap's other leg). Two,
two wire segments crossing at a right angle also connect without an
explicit junction — confirmed empirically after a CC pull-up route
crossed a pre-existing DC-DC converter trace and merged Port 4's D+
into DCDC_RAW. Both fixed by rerouting through dedicated corridors
verified against every intervening pin/wire; no unintended nets in
the final file.

Full-file check: netlist parse clean, isolation check exits 0 (only
U1/T1/CY1 bridge domains), 0 new overlaps on ports 1-3, ~14 minor
label-vs-pre-existing-text overlaps remain on Port 4 specific to that
cramped pocket (Task 4/5 content already fills most of it) — cosmetic
only, no electrical effect, left for Task 9's broader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
Parts:
- added C55, C57: 0.1uF, symbol Device:C_Small
- added C56: 22uF, symbol Device:C_Small
- added D13: TVS, symbol Device:D_TVS
- added J6: USB_C_Receptacle_USB2.0_16P, symbol Connector:USB_C_Receptacle_USB2.0_16P
- added R44: 46.4k 1%, symbol Device:R_Small
- added R45, R46: 56k, symbol Device:R_Small
- added U15: TPS2553DBV, symbol isolator-lib:TPS2553DBV
- added U19: USBLC6-2SC6, symbol Power_Protection:USBLC6-2SC6
Connections:
- net GND2: now also C55.2, C56.2, C57.2, D13.1 (A1), J6.A1 (GND), J6.A12 (GND), J6.B1 (GND), J6.B12 (GND), J6.SH (SHIELD), R44.1, U15.2 (GND), U19.2 (GND)
- net ISO_5V: now also C55.1, U15.1 (IN)
- net OCS4: now also U15.4 (~{FAULT})
- net PRTPWR4: now also U15.3 (EN)
- net PORT4_D-: now reaches U11.8 (USBDM_DN4/PRT_DIS_M4)
- net PORT4_D-: now also U19.1 (I/O1)
- net PORT4_D+: now reaches U11.9 (USBDP_DN4/PRT_DIS_P4)
- net PORT4_D+: now also U19.3 (I/O2)
- new net: J6.A5 (CC1), R45.1
- new net: R44.2, U15.5 (ILIM)
- new net: J6.A6 (D+), J6.B6 (D+), U19.4 (I/O2)
- new net: J6.A7 (D-), J6.B7 (D-), U19.6 (I/O1)
- new net: J6.B5 (CC2), R46.1
- new net PORT4_VBUS: C56.1, C57.1, D13.2 (A2), J6.A4 (VBUS), J6.A9 (VBUS), J6.B4 (VBUS), J6.B9 (VBUS), R45.2, R46.2, U15.6 (OUT), U19.5 (VBUS)
