File: hub.kicad_sch (KiCad schematic)
At the start: 141 parts, among them J1 USB_C_Receptacle_USB2.0_16P, J2 USB_C_Receptacle_PowerOnly_6P, J3 USB_A, J4 USB_A, J5 USB_C_Receptacle_USB2.0_16P, J6 USB_C_Receptacle_USB2.0_16P, Q1 2N7002, Q2 2N7002, Q3 2N7002, Q4 2N7002, T1 750313638, U1 ADuM4165, U10 TPS62203DBVR, U11 USB2514B, U12 TPS2553DBV, U13 TPS2553DBV, U14 TPS2553DBV, U15 TPS2553DBV, U16 USBLC6-2SC6, U17 USBLC6-2SC6, U18 USBLC6-2SC6, U19 USBLC6-2SC6, U2 USBLC6-2SC6, U3 TLV7042DDFR, U5 SN6505BDBV, U6 TPS630701RNM, U7 TLV7042DDFR, U8 TPS2121, Y1 24MHz, Y2 24MHz

Commit message: feat(revb/sch): Task 9 complete — CY1, PWR_FLAGs, ERC zero
CY1 (1 nF Y1-rated, 400 VAC) placed between GND1/GND2 as the sole
intentional barrier bridge, Description field documents the safety
rating. Seven PWR_FLAGs added in a dedicated corner block for every
externally-driven power net ERC couldn't otherwise resolve: GND1,
GND2, VBUS_HOST, EXT_5V, VDD1, DCDC_RAW, ISO_3V3.

ERC driven from 48 violations down to 2 (both a confirmed-benign
kicad-cli lib_symbol_mismatch quirk on TLV7042DDFR — byte-identical
content verified against the library master, re-sync doesn't clear
it). Isolation check holds: only U1, T1, CY1 bridge domains.

Along the way, fixed real bugs surfaced by driving ERC to zero
(not just silenced the warnings):

- U6 (TPS630701) PG pin was hard-wired to VOUT with no pull-up,
  directly shorting the 5V rail to GND2 whenever PG asserted. Now
  routed through R12 (100k, already present but bypassed by a wire
  that cut straight through it) per the part-selection decision
  record.
- U1 (ADuM4165) VDD2 pin was floating except for its own decoupling
  cap — merged onto the already-present ISO_3V3 rail, matching how
  VBUS2 is wired.
- U11 (USB2514B) TEST tied to GND2, PLLFILT and the second CRFILT
  bypass cap added per Microchip's official schematic checklist
  (0.01uF + 0.1uF each, PLLFILT and CRFILT kept on separate nodes
  per their explicit "do not connect" caution).
- All four TPS2553 FAULT/OCS lines were missing pull-ups entirely
  (open-drain outputs with nothing pulling them high) — added
  100k pull-ups to ISO_3V3 on all four ports.
- Y2's crystal case (pins 2/4) was floating, not tied to GND2.
- J2's external-supply CC-sensing comparator (U7/TLV7042DDFR) had
  several wires routed straight through unrelated component pins,
  shorting CC1 onto the raw EXT_5V rail, bridging two comparator
  inputs together, and tying OUTA directly to EXT_5V instead of
  the wire-OR fault node. Rebuilt to match the decision record:
  CC1/CC2 into the comparator via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
Parts:
- added C58, C60: 0.01uF, symbol Device:C_Small
- added C59: 0.1uF, symbol Device:C_Small
- added CY1: 1nF Y1, symbol Device:C_Small
- added R47, R48, R49, R50: 100k, symbol Device:R_Small
Connections:
- net VDD2 is gone; now on net ISO_3V3: C29.2, U1.18 (VDD2)
- net CRFILT_NODE: now also C60.2
- net EXT_5V: no longer C25.1, J2.A5 (CC1), R16.1, R18.2, R19.1, R20.1, U7.1 (OUTA), U7.3 (INA+)
- net GND1: now also CY1.1
- net GND2: now also U11.11 (TEST), Y2.2 (G), Y2.4 (G), C58.1, C59.1, C60.1, CY1.2
- net ISO_3V3: now also R47.2, R48.2, R49.2, R50.2
- net ISO_5V_PRE: no longer R12.2, U6.2 (PG)
- net OCS1: now also R47.1
- net OCS2: now also R48.1
- net OCS3: now also R49.1
- net OCS4: now also R50.1
- net at Q3.1 (G), R22.2, U7.7 (OUTB): now also U7.1 (OUTA)
- net at U11.34 (PLLFILT): now also C58.2, C59.2
- net at R20.2, U7.2 (INA-): no longer U7.5 (INB+)
- new net: J2.A5 (CC1), R16.1, R20.1
- new net: R12.2, U6.2 (PG)
- new net: C25.1, R18.2, R19.1, U7.3 (INA+), U7.5 (INB+)
- no-connect marks 2 -> 7
