File: hub.kicad_sch (KiCad schematic)
At the start: 149 parts, among them J1 USB_C_Receptacle_USB2.0_16P, J2 USB_C_Receptacle_PowerOnly_6P, J3 USB_A, J4 USB_A, J5 USB_C_Receptacle_USB2.0_16P, J6 USB_C_Receptacle_USB2.0_16P, Q1 2N7002, Q2 2N7002, Q3 2N7002, Q4 2N7002, T1 750313638, U1 ADuM4165, U10 TPS62203DBVR, U11 USB2514B, U12 TPS2553DBV, U13 TPS2553DBV, U14 TPS2553DBV, U15 TPS2553DBV, U16 USBLC6-2SC6, U17 USBLC6-2SC6, U18 USBLC6-2SC6, U19 USBLC6-2SC6, U2 USBLC6-2SC6, U3 TLV7042DDFR, U5 SN6505BDBV, U6 TPS630701RNM, U7 TLV7042DDFR, U8 TPS2121, Y1 24MHz, Y2 24MHz

Commit message: feat(revc): capture TI hub and hardware power protection
Parts:
- removed C1, C10, C12, C14, C23, C25, C26, C27, C28, C29, C3, C34, C35, C36, C37, C38, C39, C4, C40, C43, C45, C46, C48, C49, C51, C55, C57, C59, C7, C8: 0.1uF, symbol Device:C_Small
- removed C11, C2, C24, C41: 4.7uF, symbol Device:C_Small
- removed C13: 47uF, symbol Device:C_Small
- removed C15, C16, C30, C31: 10uF, symbol Device:C_Small
- removed C17, C21, C22: 100nF, symbol Device:C_Small
- removed C18, C19, C20, C44, C47, C50, C56: 22uF, symbol Device:C_Small
- removed C32, C33: 18pF, symbol Device:C_Small
- removed C42: 1uF, symbol Device:C_Small
- removed C5, C6: 8pF, symbol Device:C_Small
- removed C58, C60: 0.01uF, symbol Device:C_Small
- removed CY1: 1nF Y1, symbol Device:C_Small
- removed D1, D10, D13, D5, D8, D9: TVS, symbol Device:D_TVS
- removed D2, D6, D7: LED, symbol Device:LED
- removed D3, D4: SS34, symbol Device:D_Schottky
- removed J1, J5, J6: USB_C_Receptacle_USB2.0_16P, symbol Connector:USB_C_Receptacle_USB2.0_16P
- removed J2: USB_C_Receptacle_PowerOnly_6P, symbol Connector:USB_C_Receptacle_PowerOnly_6P
- removed J3, J4: USB_A, symbol Connector:USB_A
- removed L1: 1.5uH, symbol Device:L_Small
- removed L2: 10uH, symbol Device:L_Small
- removed Q1, Q2, Q3, Q4: 2N7002, symbol isolator-lib:2N7002
- removed R1, R16, R17, R2: 5.1k, symbol Device:R_Small
- removed R10: 0, symbol Device:R_Small
- removed R11, R12, R22, R31, R34, R35, R36, R37, R47, R48, R49, R5, R50: 100k, symbol Device:R_Small
- removed R13: 523k DNP, symbol Device:R_Small
- removed R14: 100k DNP, symbol Device:R_Small
- removed R15: 0 DNP, symbol Device:R_Small
- removed R18: 30.1k, symbol Device:R_Small
- removed R19: 9.76k, symbol Device:R_Small
- removed R20, R21, R28, R33, R6, R7, R8: 10k, symbol Device:R_Small
- removed R23: 17.8k, symbol Device:R_Small
- removed R24: 10.0k, symbol Device:R_Small
- removed R25: 23.7k, symbol Device:R_Small
- removed R26, R4: 10.2k, symbol Device:R_Small
- removed R27: 35.7k, symbol Device:R_Small
- removed R29: 1k, symbol Device:R_Small
- removed R3: 66.5k, symbol Device:R_Small
- removed R30, R9: 3.3k, symbol Device:R_Small
- removed R32: 12.0k 1%, symbol Device:R_Small
- removed R38, R39, R40, R44: 46.4k 1%, symbol Device:R_Small
- removed R42, R43, R45, R46: 56k, symbol Device:R_Small
- removed T1: 750313638, isolator-lib:WE_750313638, symbol isolator-lib:750313638
- removed U1: ADuM4165, symbol Isolator:ADUM4165
- removed U10: TPS62203DBVR, symbol Regulator_Switching:TPS62203DBV
- removed U11: USB2514B, symbol Interface_USB:USB2514B_Bi
- removed U12, U13, U14, U15: TPS2553DBV, symbol isolator-lib:TPS2553DBV
- removed U16, U17, U18, U19, U2: USBLC6-2SC6, symbol Power_Protection:USBLC6-2SC6
- removed U3, U7: TLV7042DDFR, symbol isolator-lib:TLV7042DDFR
- removed U5: SN6505BDBV, symbol Power_Management:SN6505BDBV
- removed U6: TPS630701RNM, symbol isolator-lib:TPS630701RNM
- removed U8: TPS2121, symbol isolator-lib:TPS2121
- removed Y1, Y2: 24MHz, symbol Device:Crystal_GND24_Small
Connections:
- no-connect marks 7 -> 0
Other:
- added sheet Downstream USB-A ports 1 and 2 (hub-ports_a.kicad_sch)
- added sheet Downstream USB-C port 3 (hub-port_c3.kicad_sch)
- added sheet Downstream USB-C port 4 (hub-port_c4.kicad_sch)
- added sheet Host USB-C input and current qualification (hub-host.kicad_sch)
- added sheet ISOUSB211 isolated 480 Mbps USB link (hub-isolation.kicad_sch)
- added sheet Isolated host power and separate shield frames (hub-converter.kicad_sch)
- added sheet Qualified external 5 V input and voltage regulation (hub-external.kicad_sch)
- added sheet Supply selection and protected port distribution (hub-distribution.kicad_sch)
- added sheet USB2514B hub, 3.3 V supply, clock and configuration (hub-hub.kicad_sch)
- note added: "Design verification in progress. PCB placement and all routing are unfinished."
- note added: "ISOLATED FOUR-PORT USB 2.0 HUB"
- note added: "ISOUSB211DPR | USB2514B | 2 x USB-A + 2 x USB-C | 480 Mbps"
- note removed: "- Comparators (U3, TLV7042) are wired INVERTING: CC -> IN-, V_REF -> IN+. Open-drain outputs OUTA/OUTB wire-OR onto"
- note removed: "- On an e-marked cable, one CC line carries VCONN at ~5 V, which reads as a false high (>0.66 V) at the unused"
- note removed: "- Q1 (2N7002) inverts CC_DET_L to drive HOST_PWR_OK active-high: gate=CC_DET_L, source=GND1, drain=HOST_PWR_OK, pulled"
- note removed: "- R_EN sizing is not a guess: SN6505B EN leakage is 20 uA max against a 0.7*VCC threshold, so R_EN <="
- note removed: "- Status LED D2 lights on INSUFFICIENT host power: Q2's gate reads CC_DET_L directly (already active-high for"
- note removed: "- The reference MUST stay on VBUS_HOST, never on an isolated rail or anything downstream of EN/HOST_PWR_OK. The"
- note removed: "- V_REF = 0.66 V, from a VBUS_HOST divider (R3/R4). This is the USB Type-C sink threshold for a 1.5 A source"
- note removed: "0.3*VBUS(min)/20uA = 71k. R6 = 10k gives EN ~4.55 V against a 3.325 V threshold (1.225 V margin). 100k here would"
- note removed: ">=1.5 A."
- note removed: "CC current-advertisement sensing (GND1) -- design notes:"
- note removed: "CC_DET_L through R5 (100k to VBUS_HOST): CC_DET_L is LOW when EITHER CC line exceeds 0.66 V (adequate host power),"
- note removed: "CP2 rule (Table 9-3): CP2=hi,PR1=lo selects IN2; CP2=PR1=lo selects VCOMP (higher wins). CP2(pin3)=STATIC bias from ISO_5V_PRE, 23.7k/10.2k to GND2, never the 3A detect."
- note removed: "HIGH otherwise."
- note removed: "OR only needs ONE CC line correct to assert. A false trigger here never asserts on a low-power host."
- note removed: "PR1(pin6)=driven by 3A-detect 2N7002 inverter, 17.8k/10.0k EXT_5V to GND2. Switchback: approx 4.18V nominal, worst-case 3.92-4.54V -- measure at bring-up."
- note removed: "Task 4: Upstream CC current-advertisement sensing (GND1)"
- note removed: "Task 6: External supply, 3A detect, TPS2121 priority mux (GND2)"
- note removed: "UPSTREAM HOST (GND1)"
- note removed: "advertisement (Rp/CC voltage band per USB-PD/Type-C spec). CC1/CC2 above this level means the host is advertising"
- note removed: "comparator input. This is benign: VCONN only appears alongside cables/sources rated for high current, and the wire-"
- note removed: "comparison result is what starts the converter; a reference derived from the converter's own output is a latch-up by"
- note removed: "construction."
- note removed: "fail (~2.75 V, below threshold)."
- note removed: "insufficient, no extra inverter needed) and sinks D2+R9 from VBUS_HOST when on."
- note removed: "up by R_EN (R6) to VBUS_HOST. HOST_PWR_OK feeds SN6505B.EN in Task 5."
- title: (none) -> Rev C — Isolated four-port USB 2.0 hub

Commit message: feat(revc): place synchronized unrouted board and correct bus startup
Other:
- sheet Downstream USB-A ports 1 and 2 renamed PORTS A
- sheet Downstream USB-C port 3 renamed PORT C3
- sheet Downstream USB-C port 4 renamed PORT C4
- sheet Host USB-C input and current qualification renamed HOST
- sheet ISOUSB211 isolated 480 Mbps USB link renamed ISOLATION
- sheet Isolated host power and separate shield frames renamed CONVERTER
- sheet Qualified external 5 V input and voltage regulation renamed EXTERNAL
- sheet Supply selection and protected port distribution renamed DISTRIBUTION
- sheet USB2514B hub, 3.3 V supply, clock and configuration renamed HUB
- added sheet BUS START (hub-bus_start.kicad_sch)
- note added: "Bus-power capacitor charging and fault timing"
- note added: "Downstream USB-A ports 1 and 2"
- note added: "Downstream USB-C port 3"
- note added: "Downstream USB-C port 4"
- note added: "Host USB-C input and current qualification"
- note added: "ISOUSB211 isolated 480 Mbps USB link"
- note added: "Isolated host power and separate shield frames"
- note added: "Qualified external 5 V input and voltage regulation"
- note added: "Supply selection and protected port distribution"
- note added: "USB2514B hub, 3.3 V supply, clock and configuration"
Changed lines of the file:
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@@
   (version 20250114)
   (generator "eeschema")
-  (paper "A3")
+  (paper "A2")
   (title_block
     (title "Rev C — Isolated four-port USB 2.0 hub")
@@
       (color 0 0 0 0)
     )
-    (property "Sheetname" "Host USB-C input and current qualification"
+    (property "Sheetname" "HOST"
       (at 20.32 53.34 0)
       (effects
@@
     )
   )
+  (text "Host USB-C input and current\nqualification"
+    (at 25.4 68.58 0)
+    (effects
+      (font
+        (size 1.524 1.524)
+      )
+      (justify left)
+    )
+  )
   (sheet
     (at 149.85999999999999 55.88)
@@
       (color 0 0 0 0)
     )
-    (property "Sheetname" "ISOUSB211 isolated 480 Mbps USB link"
+    (property "Sheetname" "ISOLATION"
       (at 149.85999999999999 53.34 0)
       (effects
@@
     )
   )
+  (text "ISOUSB211 isolated 480 Mbps USB link"
+    (at 154.94 68.58 0)
+    (effects
+      (font
+        (size 1.524 1.524)
+      )
+      (justify left)
+    )
+  )
   (sheet
     (at 279.4 55.88)
@@
       (color 0 0 0 0)
     )
-    (property "Sheetname" "Isolated host power and separate shield frames"
+    (property "Sheetname" "CONVERTER"
       (at 279.4 53.34 0)
       (effects
@@
     )
   )
+  (text "Isolated host power and separate\nshield frames"
+    (at 284.47999999999996 68.58 0)
+    (effects
+      (font
+        (size 1.524 1.524)
+      )
+      (justify left)
+    )
+  )
+  (sheet
+    (at 408.94 55.88)
+    (size 111.76 40.64)
+    (stroke
+      (width 0.254)
+      (type default)
+    )
+    (fill
+      (color 0 0 0 0)
+    )
+    (property "Sheetname" "EXTERNAL"
+      (at 408.94 53.34 0)
+      (effects
+        (font
+          (size 1.27 1.27)
+        )
+        (justify left)
+      )
+    )
+    (property "Sheetfile" "hub-external.kicad_sch"
+      (at 408.94 99.06 0)
+      (effects
+        (font
+          (size 1.27 1.27)
+        )
+        (justify left)
+      )
+    )
+    (instances
+      (project "hub"
+        (path "/c86df239-2775-4bfb-906f-796343d9aaf9"
+          (page "5")
+        )
+      )
+    )
+  )
+  (text "Qualified external 5 V input and\nvoltage regulation"
+    (at 414.02 68.58 0)
+    (effects
+      (font
+        (size 1.524 1.524)
+      )
+      (justify left)
+    )
+  )
   (sheet
     (at 20.32 119.38)
@@
       (color 0 0 0 0)
     )
-    (property "Sheetname" "Qualified external 5 V input and voltage regulation"
+    (property "Sheetname" "DISTRIBUTION"
       (at 20.32 116.83999999999999 0)
       (effects
@@
       )
     )
-    (property "Sheetfile" "hub-external.kicad_sch"
+    (property "Sheetfile" "hub-distribution.kicad_sch"
       (at 20.32 162.56 0)
       (effects
@@
       (project "hub"
         (path "/c86df239-2775-4bfb-906f-796343d9aaf9"
-          (page "5")
-        )
-      )
+          (page "6")
+        )
+      )
+    )
+  )
+  (text "Supply selection and protected port\ndistribution"
+    (at 25.4 132.07999999999998 0)
+    (effects
+      (font
+        (size 1.524 1.524)
+      )
+      (justify left)
     )
   )
@@
       (color 0 0 0 0)
     )
-    (property "Sheetname" "Supply selection and protected port distribution"
+    (property "Sheetname" "BUS START"
       (at 149.85999999999999 116.83999999999999 0)
       (effects
@@
       )
     )
-    (property "Sheetfile" "hub-distribution.kicad_sch"
+    (property "Sheetfile" "hub-bus_start.kicad_sch"
       (at 149.85999999999999 162.56 0)
       (effects
@@
       (project "hub"
         (path "/c86df239-2775-4bfb-906f-796343d9aaf9"
-          (page "6")
-        )
-      )
+          (page "7")
+        )
+      )
+    )
+  )
+  (text "Bus-power capacitor charging and\nfault timing"
+    (at 154.94 132.07999999999998 0)
+    (effects
+      (font
+        (size 1.524 1.524)
+      )
+      (justify left)
     )
   )
@@
       (color 0 0 0 0)
     )
-    (property "Sheetname" "USB2514B hub, 3.3 V supply, clock and configuration"
+    (property "Sheetname" "HUB"
       (at 279.4 116.83999999999999 0)
       (effects
@@
       (project "hub"
         (path "/c86df239-2775-4bfb-906f-796343d9aaf9"
-          (page "7")
-        )
-      )
+          (page "8")
+        )
+      )
+    )
+  )
+  (text "USB2514B hub, 3.3 V supply, clock and\nconfiguration"
+    (at 284.47999999999996 132.07999999999998 0)
+    (effects
+      (font
+        (size 1.524 1.524)
+      )
+      (justify left)
+    )
+  )
+  (sheet
+    (at 408.94 119.38)
+    (size 111.76 40.64)
+    (stroke
+      (width 0.254)
+      (type default)
+    )
+    (fill
+      (color 0 0 0 0)
+    )
+    (property "Sheetname" "PORTS A"
+      (at 408.94 116.83999999999999 0)
+      (effects
+        (font
+          (size 1.27 1.27)
+        )
+        (justify left)
+      )
+    )
+    (property "Sheetfile" "hub-ports_a.kicad_sch"
+      (at 408.94 162.56 0)
+      (effects
+        (font
+          (size 1.27 1.27)
+        )
+        (justify left)
+      )
+    )
+    (instances
+      (project "hub"
+        (path "/c86df239-2775-4bfb-906f-796343d9aaf9"
+          (page "9")
+        )
+      )
+    )
+  )
+  (text "Downstream USB-A ports 1 and 2"
+    (at 414.02 132.07999999999998 0)
+    (effects
+      (font
+        (size 1.524 1.524)
+      )
+      (justify left)
     )
   )
@@
       (color 0 0 0 0)
     )
-    (property "Sheetname" "Downstream USB-A ports 1 and 2"
+    (property "Sheetname" "PORT C3"
       (at 20.32 180.34 0)
       (effects
@@
       )
     )
-    (property "Sheetfile" "hub-ports_a.kicad_sch"
+    (property "Sheetfile" "hub-port_c3.kicad_sch"
       (at 20.32 226.06 0)
       (effects
@@
       (project "hub"
         (path "/c86df239-2775-4bfb-906f-796343d9aaf9"
-          (page "8")
-        )
-      )
+          (page "10")
+        )
+      )
+    )
+  )
+  (text "Downstream USB-C port 3"
+    (at 25.4 195.57999999999998 0)
+    (effects
+      (font
+        (size 1.524 1.524)
+      )
+      (justify left)
     )
   )
@@
       (color 0 0 0 0)
     )
-    (property "Sheetname" "Downstream USB-C port 3"
+    (property "Sheetname" "PORT C4"
       (at 149.85999999999999 180.34 0)
       (effects
@@
       )
     )
-    (property "Sheetfile" "hub-port_c3.kicad_sch"
+    (property "Sheetfile" "hub-port_c4.kicad_sch"
       (at 149.85999999999999 226.06 0)
       (effects
@@
       (project "hub"
         (path "/c86df239-2775-4bfb-906f-796343d9aaf9"
-          (page "9")
-        )
-      )
-    )
-  )
-  (sheet
-    (at 279.4 182.88)
-    (size 111.76 40.64)
-    (stroke
-      (width 0.254)
-      (type default)
-    )
-    (fill
-      (color 0 0 0 0)
-    )
-    (property "Sheetname" "Downstream USB-C port 4"
-      (at 279.4 180.34 0)
-      (effects
-        (font
-          (size 1.27 1.27)
-        )
-        (justify left)
-      )
-    )
-    (property "Sheetfile" "hub-port_c4.kicad_sch"
-      (at 279.4 226.06 0)
-      (effects
-        (font
-          (size 1.27 1.27)
-        )
-        (justify left)
-      )
-    )
-    (instances
-      (project "hub"
-        (path "/c86df239-2775-4bfb-906f-796343d9aaf9"
-          (page "10")
-        )
-      )
-    )
-  )
+          (page "11")
+        )
+      )
+    )
+  )
+  (text "Downstream USB-C port 4"
+    (at 154.94 195.57999999999998 0)
+    (effects
+      (font
+        (size 1.524 1.524)
+      )
+      (justify left)
+    )
+  )
