File: hub-bus_start.kicad_sch (KiCad schematic)
At the start: 5 parts, among them U48 SN74LVC1G17DBVR

Commit message: feat(revc): finish verified TI hub routing handoff
Parts:
- added D20, D21, D22, D23: BAT54C, hub-lib:SOT-23, symbol hub-lib:Diode_BAT54C
- added D6: GREEN, hub-lib:LED_0603_1608Metric, symbol hub-lib:Device_LED
- added Q3: 2N7002, hub-lib:SOT-23, symbol hub-lib:Transistor_FET_2N7002
- added R29: 3.3kR, hub-lib:R_0402_1005Metric, symbol hub-lib:Device_R_Small_US
- R121: value 47kR -> 68kR; LCSC (none) -> C77607; MPN ERJ2RKF4702X -> ERJ2RKF6802X
Connections:
- net GND2: now also Q3.2 (S)
- net ISO_3V3: now also R29.1
- net PORT_LIMIT_N: now also D20.3, D21.3
- new net D6_A: D6.2 (A), R29.2
- new net D6_K: D6.1 (K), Q3.3 (D)
- new net EXT_SELECTED: Q3.1 (G)
- new net OCS1_N: D20.1, D22.1
- new net OCS2_N: D20.2, D22.2
- new net OCS3_N: D21.1, D23.1
- new net OCS4_N: D21.2, D23.2
- new net PORT_RAIL_OK: D22.3, D23.3
Other:
- note added: "Aggregate fault fanout and external-source indicator"
- note added: "Bus startup and aggregate fault reporting"
- note added: "Delayed bus fault report; immediate current limit"
- note added: "USB 2.0 / 480 Mbps | Rev C electrical design | Placed PCB; all routing by Alex; hardware tests pending"
- note removed: "Bus current limit is immediate; report sustained faults after capacitor charging"
- note removed: "Bus-power capacitor charging and fault timing"
- note removed: "USB 2.0 / 480 Mbps | Rev C electrical design | Placement and routing review pending"
- title: Bus-power capacitor charging and fault timing -> Bus startup and aggregate fault reporting
