File: hub-converter.kicad_sch (KiCad schematic)
At the start: 27 parts, among them T1 750313638, U5 SN6505BDBVR, U6 TPS630701RNMR

Commit message: feat(revc): assign exact BOM and verified local land patterns
Parts:
- C10, C12, C14, C17, C21, C22: footprint (none) -> hub-lib:C_0402_1005Metric; LCSC (none) -> C77020; MPN (none) -> GRM155R71H104KE14D; Manufacturer (none) -> Murata Manufacturing; Ratings (none) -> 50V X7R 10%
- C11: footprint (none) -> hub-lib:C_0603_1608Metric; LCSC (none) -> C90057; MPN (none) -> GRM188R61E475KE11D; Manufacturer (none) -> Murata Manufacturing; Ratings (none) -> 25V X5R 10%
- C13, C15, C16, C18, C19, C20: footprint (none) -> hub-lib:C_1210_3225Metric; LCSC (none) -> C21397; MPN (none) -> GRM32ER71E226KE15L; Manufacturer (none) -> Murata Manufacturing; Ratings (none) -> 25V X7R 10%
- D3, D4: footprint Diode_SMD:D_SMA -> hub-lib:D_SMA; LCSC (none) -> C8678; Ratings (none) -> See exact manufacturer datasheet
- L1: footprint (none) -> hub-lib:Coilcraft_XFL4020_4x4mm; LCSC (none) -> C3033018; Ratings (none) -> See exact manufacturer datasheet
- R10, R15: footprint (none) -> hub-lib:R_0402_1005Metric; LCSC (none) -> C242160; MPN (none) -> ERJ2GE0R00X; Manufacturer (none) -> Panasonic Industry; Ratings (none) -> 0R jumper, 0402, 1A rated current
- R11, R12: footprint (none) -> hub-lib:R_0402_1005Metric; LCSC (none) -> C192169; MPN (none) -> ERJ2RKF1003X; Manufacturer (none) -> Panasonic Industry; Ratings (none) -> 1%, 0.1W, 50V
- SH1: footprint (none) -> hub-lib:Laird_Technologies_BMI-S-201-F_13.66x12.70mm; CoverMPN (none) -> BMI-S-201-C; CoverQuantity (none) -> 1; Ratings (none) -> Separate grounded frame; removable BMI-S-201-C ordered sepa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
- SH2: footprint (none) -> hub-lib:Laird_Technologies_BMI-S-209-F_29.36x18.50mm; CoverMPN (none) -> BMI-S-209-C; CoverQuantity (none) -> 1; Ratings (none) -> Separate grounded frame; removable BMI-S-209-C ordered sepa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
- T1: footprint isolator-lib:WE_750313638 -> hub-lib:WE_750313638; Ratings (none) -> See exact manufacturer datasheet
- TP5, TP6: footprint TestPoint:TestPoint_Pad_D1.0mm -> hub-lib:TestPoint_Pad_D1.0mm; Manufacturer (none) -> PCB feature; Ratings (none) -> Exposed test pad; no purchased part; now left out of the parts list
- U5: footprint (none) -> hub-lib:SOT-23-6; LCSC (none) -> C74518; Ratings (none) -> See exact manufacturer datasheet
- U6: footprint (none) -> hub-lib:TPS630701RNM_VQFN-HR-15; LCSC (none) -> C2876599; Ratings (none) -> See exact manufacturer datasheet

Commit message: feat(revc): place synchronized unrouted board and correct bus startup
Other:
- note added: "Declared power origins"
- note added: "Isolated 5 V regulation"
- note added: "Primary push-pull driver and transformer"
- note added: "Secondary rectifier and reservoir"
- note added: "Two separate shield frames"
- note added: "USB 2.0 / 480 Mbps | Rev C electrical design | Placement and routing review pending"
- note removed: "Rev C | all routing reserved for Alex | electrical draft under review"
- moved on the sheet: C10, C11, C12, C13, C14, C15, C16, C17, C18, C19, C20, C21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

Commit message: feat(revc): finish verified TI hub routing handoff
Other:
- note added: "USB 2.0 / 480 Mbps | Rev C electrical design | Placed PCB; all routing by Alex; hardware tests pending"
- note removed: "USB 2.0 / 480 Mbps | Rev C electrical design | Placement and routing review pending"
- moved on the sheet: D3, D4, TP5
