File: hub-distribution.kicad_sch (KiCad schematic)
At the start: 49 parts, among them Q3 2N7002, U29 TPS2553DBVR-1, U30 TPS22975NDSGR, U31 TPS3808G01DBVR, U32 SN74LVC1G08DBVR, U41 SN74LVC1G08DBVR, U42 SN74LVC1G04DBVR, U43 SN74LVC1G08DBVR, U47 INA300AIDGSR, U8 TPS2121RUXR

Commit message: feat(revc): assign exact BOM and verified local land patterns
Parts:
- C107, C108, C109, C112, C27, C93, C94, C95, C96, C97: footprint (none) -> hub-lib:C_0402_1005Metric; LCSC (none) -> C77020; MPN (none) -> GRM155R71H104KE14D; Manufacturer (none) -> Murata Manufacturing; Ratings (none) -> 50V X7R 10%
- C115: footprint (none) -> hub-lib:C_0402_1005Metric; LCSC (none) -> C77023; MPN (none) -> GRM155R71H223KA12D; Manufacturer (none) -> Murata Manufacturing; Ratings (none) -> 50V X7R 10%
- C92: footprint (none) -> hub-lib:CP_Elec_8x6.2; LCSC (none) -> C401648; MPN (none) -> EEEFK1A221P; Manufacturer (none) -> Panasonic Industry; Ratings (none) -> 220uF 10V +/-20%; 8mm diameter, 6.5mm maximum height; polar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
- D14, D15, D16, D17: footprint Diode_SMD:D_SOD-323 -> hub-lib:D_SOD-323; LCSC (none) -> C124205; Ratings (none) -> See exact manufacturer datasheet
- D20, D21, D22, D23: footprint Package_TO_SOT_SMD:SOT-23 -> hub-lib:SOT-23; LCSC (none) -> C37704; Ratings (none) -> See exact manufacturer datasheet
- D6: footprint LED_SMD:LED_0603_1608Metric -> hub-lib:LED_0603_1608Metric; LCSC (none) -> C125094; Ratings (none) -> See exact manufacturer datasheet
- Q3: footprint Package_TO_SOT_SMD:SOT-23 -> hub-lib:SOT-23; LCSC (none) -> C65189; Ratings (none) -> See exact manufacturer datasheet
- R116: footprint (none) -> hub-lib:R_1206_3216Metric; LCSC (none) -> C844910; MPN (none) -> WSLP1206R0100FEA; Manufacturer (none) -> Vishay; Ratings (none) -> 1W, 1%, 75ppm/C; Kelvin sense
- R117: footprint (none) -> hub-lib:R_0603_1608Metric; LCSC (none) -> C860186; MPN (none) -> RT0603BRB071K1L; Manufacturer (none) -> Yageo; Ratings (none) -> 0.1%, 10ppm/C thin film, 0.1W
- R23: footprint (none) -> hub-lib:R_0402_1005Metric; MPN (none) -> ERJ2RKF1782X; Manufacturer (none) -> Panasonic Industry; Ratings (none) -> 1%, 0.1W, 50V
- R24, R28, R63, R66, R83: footprint (none) -> hub-lib:R_0402_1005Metric; LCSC (none) -> C191123; MPN (none) -> ERJ2RKF1002X; Manufacturer (none) -> Panasonic Industry; Ratings (none) -> 1%, 0.1W, 50V
- R25: footprint (none) -> hub-lib:R_0402_1005Metric; MPN (none) -> ERJ2RKF2372X; Manufacturer (none) -> Panasonic Industry; Ratings (none) -> 1%, 0.1W, 50V
- R26: footprint (none) -> hub-lib:R_0402_1005Metric; LCSC (none) -> C2076944; MPN (none) -> ERJ2RKF1022X; Manufacturer (none) -> Panasonic Industry; Ratings (none) -> 1%, 0.1W, 50V
- R27: footprint (none) -> hub-lib:R_0402_1005Metric; MPN (none) -> ERJ2RKF2982X; Manufacturer (none) -> Panasonic Industry; Ratings (none) -> 1%, 0.1W, 50V
- R29: footprint (none) -> hub-lib:R_0402_1005Metric; LCSC (none) -> C409909; MPN (none) -> ERJ2RKF3301X; Manufacturer (none) -> Panasonic Industry; Ratings (none) -> 1%, 0.1W, 50V
- R62: footprint (none) -> hub-lib:R_0402_1005Metric; LCSC (none) -> C413105; MPN (none) -> ERJ2RKF7502X; Manufacturer (none) -> Panasonic Industry; Ratings (none) -> 1%, 0.1W, 50V
- R64: footprint (none) -> hub-lib:R_0603_1608Metric; LCSC (none) -> C860056; MPN (none) -> RT0603BRB07100KL; Manufacturer (none) -> Yageo; Ratings (none) -> 0.1%, 10ppm/C thin film, 0.1W
- R65: footprint (none) -> hub-lib:R_0603_1608Metric; LCSC (none) -> C860067; MPN (none) -> RT0603BRB0710KL; Manufacturer (none) -> Yageo; Ratings (none) -> 0.1%, 10ppm/C thin film, 0.1W
- TP10, TP11, TP9: footprint TestPoint:TestPoint_Pad_D1.0mm -> hub-lib:TestPoint_Pad_D1.0mm; Manufacturer (none) -> PCB feature; Ratings (none) -> Exposed test pad; no purchased part; now left out of the parts list
- U29: footprint (none) -> hub-lib:SOT-23-6; LCSC (none) -> C111738; Ratings (none) -> See exact manufacturer datasheet
- U30: footprint (none) -> hub-lib:Texas_DSG0008A_WSON-8-1EP_2x2mm_P0.5mm_EP0.9x1.6mm; LCSC (none) -> C2149871; Ratings (none) -> See exact manufacturer datasheet
- U31: footprint (none) -> hub-lib:SOT-23-6; LCSC (none) -> C19653; Ratings (none) -> See exact manufacturer datasheet
- U32, U41, U43: footprint (none) -> hub-lib:SOT-23-5; LCSC (none) -> C7666; Ratings (none) -> See exact manufacturer datasheet
- U42: footprint (none) -> hub-lib:SOT-23-5; LCSC (none) -> C7827; Ratings (none) -> See exact manufacturer datasheet
- U47: footprint (none) -> hub-lib:MSOP-10_3x3mm_P0.5mm; LCSC (none) -> C529558; Ratings (none) -> See exact manufacturer datasheet
- U8: footprint (none) -> hub-lib:TI_RUX0012A_VQFN-HR12_2x2.5mm; LCSC (none) -> C485916; Ratings (none) -> See exact manufacturer datasheet

Commit message: feat(revc): place synchronized unrouted board and correct bus startup
Parts:
- U29: value TPS2553DBVR-1 -> TPS2553DBVR; LCSC C111738 -> C55266; MPN TPS2553DBVR-1 -> TPS2553DBVR
Connections:
- net PORT_LIMIT_N: no longer R63.2, U29.4 (~{FAULT})
- new net BUS_LIMIT_RAW_N: R63.2, U29.4 (~{FAULT})
Other:
- note added: "Aggregate fault fanout and source indicator"
- note added: "Bus / external downstream supply paths"
- note added: "Core undervoltage sheds downstream loads"
- note added: "Declared power origins"
- note added: "External-priority power mux and core hold-up"
- note added: "Mutually exclusive supply enables"
- note added: "USB 2.0 / 480 Mbps | Rev C electrical design | Placement and routing review pending"
- note removed: "Rev C | all routing reserved for Alex | electrical draft under review"
- moved on the sheet: C107, C108, C109, C112, C115, C27, C92, C93, C94, C95, C96, C97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

Commit message: feat(revc): finish verified TI hub routing handoff
Parts:
- removed D20, D21, D22, D23: BAT54C, hub-lib:SOT-23, symbol hub-lib:Diode_BAT54C
- removed D6: GREEN, hub-lib:LED_0603_1608Metric, symbol hub-lib:Device_LED
- removed Q3: 2N7002, hub-lib:SOT-23, symbol hub-lib:Transistor_FET_2N7002
- removed R29: 3.3kR, hub-lib:R_0402_1005Metric, symbol hub-lib:Device_R_Small_US
Other:
- note added: "USB 2.0 / 480 Mbps | Rev C electrical design | Placed PCB; all routing by Alex; hardware tests pending"
- note removed: "Aggregate fault fanout and source indicator"
- note removed: "USB 2.0 / 480 Mbps | Rev C electrical design | Placement and routing review pending"
- moved on the sheet: D14, D15, D16, D17
