File: hub-isolation.kicad_sch (KiCad schematic)
At the start: 30 parts, among them U1 ISOUSB211DPR

Commit message: feat(revc): assign exact BOM and verified local land patterns
Parts:
- C28, C3, C64: footprint (none) -> hub-lib:C_0603_1608Metric; LCSC (none) -> C77046; MPN (none) -> GRM188R61E105KA12D; Manufacturer (none) -> Murata Manufacturing; Ratings (none) -> 25V X5R 10%
- C29, C4, C63, C66, C69, C72, C75: footprint (none) -> hub-lib:C_0402_1005Metric; LCSC (none) -> C77020; MPN (none) -> GRM155R71H104KE14D; Manufacturer (none) -> Murata Manufacturing; Ratings (none) -> 50V X7R 10%
- C65, C68, C71, C74: footprint (none) -> hub-lib:C_0603_1608Metric; LCSC (none) -> C90057; MPN (none) -> GRM188R61E475KE11D; Manufacturer (none) -> Murata Manufacturing; Ratings (none) -> 25V X5R 10%
- C67, C70, C73, C76: footprint (none) -> hub-lib:C_0402_1005Metric; LCSC (none) -> C77019; MPN (none) -> GRM155R71H103KA88D; Manufacturer (none) -> Murata Manufacturing; Ratings (none) -> 50V X7R 10%
- CY1: footprint isolator-lib:C_Disc_D7.0mm_W5.5mm_P14.00mm -> hub-lib:C_Disc_D7.0mm_W5.5mm_P14.00mm; LCSC (none) -> C2914611; Ratings (none) -> See exact manufacturer datasheet
- R51, R52, R53, R54, R55, R56, R57, R58: footprint (none) -> hub-lib:R_0402_1005Metric; LCSC (none) -> C242160; MPN (none) -> ERJ2GE0R00X; Manufacturer (none) -> Panasonic Industry; Ratings (none) -> 0R jumper, 0402, 1A rated current
- TP3, TP4: footprint TestPoint:TestPoint_Pad_D1.0mm -> hub-lib:TestPoint_Pad_D1.0mm; Manufacturer (none) -> PCB feature; Ratings (none) -> Exposed test pad; no purchased part; now left out of the parts list
- U1: LCSC (none) -> C5772877; Ratings (none) -> See exact manufacturer datasheet

Commit message: feat(revc): place synchronized unrouted board and correct bus startup
Other:
- note added: "Equalization rework: fit only one strap per input"
- note added: "Host-side supply bypass: GND1 only"
- note added: "Isolated USB link: no external clock"
- note added: "Isolated-side supply bypass: GND2 only"
- note added: "Only intentional inter-ground capacitance"
- note added: "USB 2.0 / 480 Mbps | Rev C electrical design | Placement and routing review pending"
- note removed: "Rev C | all routing reserved for Alex | electrical draft under review"
- moved on the sheet: C28, C29, C3, C4, C63, C64, C65, C66, C67, C68, C69, C70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

Commit message: feat(revc): finish verified TI hub routing handoff
Other:
- note added: "USB 2.0 / 480 Mbps | Rev C electrical design | Placed PCB; all routing by Alex; hardware tests pending"
- note removed: "USB 2.0 / 480 Mbps | Rev C electrical design | Placement and routing review pending"
Changed lines of the file:
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@@
     )
   )
-  (text "USB 2.0 / 480 Mbps  |  Rev C electrical design  |  Placement and routing review pending"
+  (text "USB 2.0 / 480 Mbps  |  Rev C electrical design  |  Placed PCB; all routing by Alex; hardware tests pending"
     (at 20.32 27.94 0)
     (effects
@@
     )
   )
-  (symbol
-    (lib_id "hub-lib:power_U1_3V3_HOST")
+  (global_label "U1_3V3_HOST"
+    (shape bidirectional)
     (at 355.6 196.85 0)
-    (unit 1)
-    (in_bom no)
-    (on_board no)
-    (dnp no)
-    (property "Reference" "#PWR3022"
+    (effects
+      (font
+        (size 1.27 1.27)
+      )
+      (justify right)
+    )
+    (property "Intersheetrefs" "${INTERSHEET_REFS}"
       (at 355.6 196.85 0)
       (effects
@@
       )
     )
-    (property "Value" "U1_3V3_HOST"
-      (at 355.6 193.04 0)
-      (effects
-        (font
-          (size 1.016 1.016)
-        )
-      )
-    )
-    (pin "1"
-    )
-    (instances
-      (project "hub"
-        (path "/c86df239-2775-4bfb-906f-796343d9aaf9/792be433-2b74-58de-babf-a6aef3017e56"
-          (reference "#PWR3022")
-          (unit 1)
-        )
-      )
-    )
   )
   (symbol
@@
     (on_board no)
     (dnp no)
-    (property "Reference" "#PWR3023"
+    (property "Reference" "#PWR3022"
       (at 388.62 196.85 0)
       (effects
@@
       (project "hub"
         (path "/c86df239-2775-4bfb-906f-796343d9aaf9/792be433-2b74-58de-babf-a6aef3017e56"
-          (reference "#PWR3023")
+          (reference "#PWR3022")
           (unit 1)
         )
@@
     )
   )
-  (symbol
-    (lib_id "hub-lib:power_U1_3V3_HOST")
+  (global_label "U1_3V3_HOST"
+    (shape bidirectional)
     (at 421.64 196.85 0)
-    (unit 1)
-    (in_bom no)
-    (on_board no)
-    (dnp no)
-    (property "Reference" "#PWR3024"
+    (effects
+      (font
+        (size 1.27 1.27)
+      )
+      (justify right)
+    )
+    (property "Intersheetrefs" "${INTERSHEET_REFS}"
       (at 421.64 196.85 0)
       (effects
@@
       )
     )
-    (property "Value" "U1_3V3_HOST"
-      (at 421.64 193.04 0)
-      (effects
-        (font
-          (size 1.016 1.016)
-        )
-      )
-    )
-    (pin "1"
-    )
-    (instances
-      (project "hub"
-        (path "/c86df239-2775-4bfb-906f-796343d9aaf9/792be433-2b74-58de-babf-a6aef3017e56"
-          (reference "#PWR3024")
-          (unit 1)
-        )
-      )
-    )
   )
   (symbol
@@
     (on_board no)
     (dnp no)
-    (property "Reference" "#PWR3025"
+    (property "Reference" "#PWR3023"
       (at 454.66 196.85 0)
       (effects
@@
       (project "hub"
         (path "/c86df239-2775-4bfb-906f-796343d9aaf9/792be433-2b74-58de-babf-a6aef3017e56"
-          (reference "#PWR3025")
+          (reference "#PWR3023")
           (unit 1)
         )
@@
     )
   )
-  (symbol
-    (lib_id "hub-lib:power_ISO_3V3")
+  (global_label "ISO_3V3"
+    (shape bidirectional)
     (at 487.68 196.85 0)
-    (unit 1)
-    (in_bom no)
-    (on_board no)
-    (dnp no)
-    (property "Reference" "#PWR3026"
+    (effects
+      (font
+        (size 1.27 1.27)
+      )
+      (justify right)
+    )
+    (property "Intersheetrefs" "${INTERSHEET_REFS}"
       (at 487.68 196.85 0)
       (effects
@@
       )
     )
-    (property "Value" "ISO_3V3"
-      (at 487.68 193.04 0)
-      (effects
-        (font
-          (size 1.016 1.016)
-        )
-      )
-    )
-    (pin "1"
-    )
-    (instances
-      (project "hub"
-        (path "/c86df239-2775-4bfb-906f-796343d9aaf9/792be433-2b74-58de-babf-a6aef3017e56"
-          (reference "#PWR3026")
-          (unit 1)
-        )
-      )
-    )
   )
   (symbol
@@
     (on_board no)
     (dnp no)
-    (property "Reference" "#PWR3027"
+    (property "Reference" "#PWR3024"
       (at 520.7 196.85 0)
       (effects
@@
       (project "hub"
         (path "/c86df239-2775-4bfb-906f-796343d9aaf9/792be433-2b74-58de-babf-a6aef3017e56"
-          (reference "#PWR3027")
+          (reference "#PWR3024")
           (unit 1)
         )
@@
     )
   )
-  (symbol
-    (lib_id "hub-lib:power_ISO_3V3")
+  (global_label "ISO_3V3"
+    (shape bidirectional)
     (at 553.72 196.85 0)
-    (unit 1)
-    (in_bom no)
-    (on_board no)
-    (dnp no)
-    (property "Reference" "#PWR3028"
+    (effects
+      (font
+        (size 1.27 1.27)
+      )
+      (justify right)
+    )
+    (property "Intersheetrefs" "${INTERSHEET_REFS}"
       (at 553.72 196.85 0)
       (effects
@@
       )
     )
-    (property "Value" "ISO_3V3"
-      (at 553.72 193.04 0)
-      (effects
-        (font
-          (size 1.016 1.016)
-        )
-      )
-    )
-    (pin "1"
-    )
-    (instances
-      (project "hub"
-        (path "/c86df239-2775-4bfb-906f-796343d9aaf9/792be433-2b74-58de-babf-a6aef3017e56"
-          (reference "#PWR3028")
-          (unit 1)
-        )
-      )
-    )
   )
   (text "Only intentional inter-ground capacitance"
@@
     (dnp no)
     (property "Reference" "CY1"
-      (at 30.480000000000004 214.63 0)
+      (at 30.480000000000004 214.63 90)
       (effects
         (font
@@
     )
     (property "Value" "1nF Y1"
-      (at 30.480000000000004 217.17000000000002 0)
+      (at 30.480000000000004 217.17000000000002 90)
       (effects
         (font
