File: v1/isolator-v1.kicad_sch (KiCad schematic)
At the start: 0 parts

Commit message: feat(v1/sch): upstream USB-C host section, ADuM Side 1, crystal
Places and wires everything on the host side of the isolation barrier: J1
(USB-C receptacle), U1 (ADuM4165, Side 1 pins only, Side 2 no-connected for
Tasks 4/5), U2 (USBLC6-2SC6 D+/D- ESD), Y1 (24MHz crystal + C1/C2 load caps),
D5 (new T6V0S5A-7 VBUS TVS), R1/R2 (dedicated 5.1k CC pulldowns), C3 (4.7uF,
not v2's 10uF, to leave headroom under the USB 10uF/50uC bus-power limit),
C4/C5 (VBUS_HOST/VDD1 bypass).

Lifted lib_symbols and symbol instances verbatim from isolator.kicad_sch
(v2) wherever v2 already had the same subcircuit -- same refdes, same sheet
coordinates, regenerated UUIDs -- since v2's host-side wiring already uses
the exact net names this task needs (VBUS_HOST, HOST_D+, HOST_D-, VDD1,
XTALIN, XTALOUT, GND1). Programmatic connectivity analysis (union-find over
wire endpoints + library pin tables) separated GND1-domain content to keep
from GND2/isolated-side content to exclude. D5 and the U1 pins 11-20
no-connect markers are the only genuinely new elements.

Added 3 PWR_FLAGs (GND1, VBUS_HOST, VDD1) in a dedicated corner box to
satisfy this project's power_pin_not_driven ERC rule.

ERC: 0 violations, exit 0. Netlist probes for HOST_D+/VBUS_HOST/VDD1 match
the brief's wiring table exactly. Full verification trail and layout
coordinates for Task 4 in task-3-report.md.
Parts:
- added C1, C2: 8p, Capacitor_SMD:C_0603_1608Metric, symbol Device:C_Small
- added C3: 4.7uF, Capacitor_SMD:C_0805_2012Metric, symbol Device:C_Small
- added C4, C5: 100n, Capacitor_SMD:C_0603_1608Metric, symbol Device:C_Small
- added D5: T6V0S5A-7, Diode_SMD:D_SOD-523, symbol Device:D_TVS
- added J1: HOST, Connector_USB:USB_C_Receptacle_HRO_TYPE-C-31-M-12, symbol Connector:USB_C_Receptacle_USB2.0_16P
- added R1, R2: 5.1k, Resistor_SMD:R_0603_1608Metric, symbol Device:R_Small
- added U1: ADuM4165, isolator-lib:ADI_SOIC_IC_20_RI-20-1, symbol Isolator:ADUM4165
- added U2: USBLC6-2SC6, Package_TO_SOT_SMD:SOT-23-6, symbol Power_Protection:USBLC6-2SC6
- added Y1: 24M 8pF, Crystal:Crystal_SMD_3225-4Pin_3.2x2.5mm, symbol Device:Crystal_GND24_Small
Connections:
- new net: J1.B5 (CC2), R2.1
- new net: J1.A5 (CC1), R1.1
- new net GND1: C1.2, C2.2, C3.2, C4.2, C5.2, D5.1 (A1), J1.A1 (GND), J1.A12 (GND), J1.B1 (GND), J1.B12 (GND), J1.SH (SHIELD), R1.2, R2.2, U1.10 (GND1), U1.2 (GND1), U1.4 (GND1), U1.7 (GND1), U2.2 (GND), Y1.2 (G), Y1.4 (G)
- new net GND2: U1.11 (GND2), U1.15 (GND2), U1.16 (GND2), U1.17 (GND2), U1.19 (GND2)
- new net HOST_D+: J1.A6 (D+), J1.B6 (D+), U1.8 (UD+), U2.1 (I/O1), U2.6 (I/O1)
- new net HOST_D-: J1.A7 (D-), J1.B7 (D-), U1.9 (UD-), U2.3 (I/O2), U2.4 (I/O2)
- new net VBUS_HOST: C3.1, C4.1, D5.2 (A2), J1.A4 (VBUS), J1.A9 (VBUS), J1.B4 (VBUS), J1.B9 (VBUS), U1.1 (VBUS1), U2.5 (VBUS)
- new net VDD1: C5.1, U1.3 (VDD1)
- new net XTALIN: C1.1, U1.5 (XI1), Y1.1
- new net XTALOUT: C2.1, U1.6 (XO1), Y1.3
- no-connect marks 0 -> 9
Other:
- note added: "ISOLATOR U1 (ADuM4165) -- HOST SIDE (GND1)"
- note added: "POWER FLAGS"
- note added: "USB-C HOST PORT (GND1)"

Commit message: fix(v1/sch): Task 3 review round 1 - D5 polarity, GND2 no-connect, VDD1 typing
Critical: D5 (VBUS TVS) was wired backwards. T6V0S5A-7 datasheet and KiCad's
Device:D convention both confirm pin 1 = cathode, pin 2 = anode; my original
placement had pin 1 on GND1 and pin 2 on VBUS_HOST, forward-biasing the diode
continuously at 5V. Swapped which net each pin lands on so pin 1 -> VBUS_HOST,
pin 2 -> GND1, and corrected the symbol's Description property to match.

Important: removed the no_connect markers from U1's GND2 pins (11, 15, 16,
17, 19) -- they self-connect via KiCad's same-name hidden-power-pin rule, so
marking them no_connect was a real contradiction (ERC's no_connect_connected
warning was correct). This exposed a legitimate power_pin_not_driven error on
the now-visible GND2 net, so added a 4th PWR_FLAG (GND2) in the POWER FLAGS
corner, consistent with the existing GND1/VBUS_HOST/VDD1 pattern -- GND2 is a
real net Task 4/5 will build out, not a workaround.

Important: read the ADuM4165 datasheet's Power Supply Options section and
confirmed VDD1 is the internal LDO's output in v1's topology (VBUS1 fed from
host, nothing external drives VDD1). Retyped pin 3 in the embedded ADUM4165
symbol from power_in to power_out and removed the now-unnecessary VDD1
PWR_FLAG. Recorded the same open question for VDD2/Task 5 rather than
re-deriving it there.

ERC clean both with and without --severity-error (0 errors, 0 warnings).
Netlist confirms D5's corrected polarity and GND2's isolated cluster. Full
trail in task-3-report.md "Fix round 1".
Connections:
- net GND1: now also D5.2 (A2); no longer D5.1 (A1)
- net VBUS_HOST: now also D5.1 (A1); no longer D5.2 (A2)
- no-connect marks 9 -> 7
Changed lines of the file:
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@@
 			)
 		)
-		(property "Description" "Unidirectional TVS, VBUS ESD/surge protection, cathode->VBUS_HOST, anode->GND1"
+		(property "Description" "Unidirectional TVS, VBUS ESD/surge protection, pin1(cathode)->VBUS_HOST, pin2(anode)->GND1"
 			(at 33.02 27.94 0)
 			(hide yes)
@@
 	(symbol
 		(lib_id "power:GND1")
-		(at 29.21 34.29 0)
+		(at 36.83 34.29 0)
 		(unit 1)
 		(body_style 1)
@@
 		(fields_autoplaced yes)
 		(property "Reference" "#PWR09"
-			(at 29.21 27.94 0)
+			(at 36.83 27.94 0)
 			(show_name no)
 			(do_not_autoplace no)
@@
 		)
 		(property "Value" "GND1"
-			(at 29.21 30.48 0)
+			(at 36.83 30.48 0)
 			(show_name no)
 			(do_not_autoplace no)
@@
 		)
 		(property "Footprint" ""
-			(at 29.21 34.29 0)
+			(at 36.83 34.29 0)
 			(show_name no)
 			(do_not_autoplace no)
@@
 		)
 		(property "Datasheet" ""
-			(at 29.21 34.29 0)
+			(at 36.83 34.29 0)
 			(show_name no)
 			(do_not_autoplace no)
@@
 		)
 		(property "Description" "Power symbol creates a global label with name \"GND1\" , ground"
-			(at 29.21 34.29 0)
+			(at 36.83 34.29 0)
 			(show_name no)
 			(do_not_autoplace no)
@@
 	)
 	(label "VBUS_HOST"
-		(at 36.83 34.29 90)
+		(at 29.21 34.29 90)
 		(effects
 			(font
@@
 	)
 	(no_connect
-		(at 317.5 80.01)
-	)
-	(no_connect
-		(at 320.04 80.01)
-	)
-	(no_connect
 		(at 325.12 67.31)
 	)
@@
 	(no_connect
 		(at 317.5 46.99)
+	)
+	(wire
+		(pts
+			(xy 317.5 80.01) (xy 317.5 88.9)
+		)
+		(stroke
+			(width 0)
+			(type default)
+		)
+	)
+	(wire
+		(pts
+			(xy 317.5 88.9) (xy 320.04 88.9)
+		)
+		(stroke
+			(width 0)
+			(type default)
+		)
+	)
+	(label "GND2"
+		(at 320.04 88.9 0)
+		(effects
+			(font
+				(size 1.27 1.27)
+			)
+			(justify left bottom)
+		)
 	)
 	(rectangle
@@
 	(symbol
 		(lib_id "power:PWR_FLAG")
-		(at 81.28 247.65 0)
+		(at 106.68 247.65 0)
 		(unit 1)
 		(body_style 1)
@@
 		(dnp no)
 		(fields_autoplaced yes)
-		(property "Reference" "#FLG03"
-			(at 81.28 241.3 0)
+		(property "Reference" "#FLG04"
+			(at 106.68 241.3 0)
 			(hide yes)
 			(show_name no)
@@
 		)
 		(property "Value" "PWR_FLAG"
-			(at 83.82 246.38 0)
+			(at 109.22 246.38 0)
 			(show_name no)
 			(do_not_autoplace no)
@@
 		)
 		(property "Footprint" ""
-			(at 81.28 247.65 0)
+			(at 106.68 247.65 0)
 			(hide yes)
 			(show_name no)
@@
 		)
 		(property "Datasheet" ""
-			(at 81.28 247.65 0)
+			(at 106.68 247.65 0)
 			(hide yes)
 			(show_name no)
@@
 		)
 		(property "Description" "Special symbol for telling ERC where power comes from"
-			(at 81.28 247.65 0)
+			(at 106.68 247.65 0)
 			(hide yes)
 			(show_name no)
@@
 			(project "isolator-v1"
 				(path "/00000000-0000-0000-0000-000000000001"
-					(reference "#FLG03")
+					(reference "#FLG04")
 					(unit 1)
 				)
@@
 	(wire
 		(pts
-			(xy 81.28 247.65) (xy 81.28 255.27)
-		)
-		(stroke
-			(width 0)
-			(type default)
-		)
-	)
-	(label "VDD1"
-		(at 81.28 255.27 90)
+			(xy 106.68 247.65) (xy 106.68 255.27)
+		)
+		(stroke
+			(width 0)
+			(type default)
+		)
+	)
+	(label "GND2"
+		(at 106.68 255.27 90)
 		(effects
 			(font
